File: pcb/_autosave-pcb.kicad_pcb (KiCad board)
At the start: 2 copper layers, 205 parts, among them J1 USB_C_Receptacle_USB2.0_16P, J2 Conn_01x04, J3 Conn_01x05, U1 XC6206PxxxMR, U2 SRV05-4, U3 RP2040, U4 W25Q128JVS, Y1 Crystal_GND24

Commit message: sob
Parts:
- R7, R8, R9: moved to F.Cu
- moved J2 269.1 mm to (50.0, 39.5), turned to 90 degrees
- moved U2 267.3 mm to (43.5, 25.0)
- moved R2 258.7 mm to (40.5, 24.0), turned to 180 degrees
- moved R1 253.2 mm to (46.5, 24.0)
- moved F1 251.3 mm to (39.0, 28.5), turned to -90 degrees
- moved J1 228.1 mm to (43.5, 17.5), turned to 180 degrees
- moved J3 81.1 mm to (160.5, 208.9)
- moved C12 70.2 mm to (144.5, 214.5), turned to 135 degrees
- moved C11 69.9 mm to (144.5, 211.5), turned to -135 degrees
- moved Y1 30.0 mm to (146.3, 212.9), turned to 45 degrees
- moved R9 4.09 mm to (148.0, 214.5), turned to 45 degrees
- moved C5 1.00 mm to (137.0, 203.5)
- moved R7 1.00 mm to (146.6, 198.3)
- moved R8 1.00 mm to (147.6, 198.3)
Connections:
- U2 pad 3: D- -> unconnected-(U2-IO2-Pad3)
- U2 pad 6: unconnected-(U2-IO4-Pad6) -> D-
