File: pcb/_autosave-pcb.kicad_pcb (KiCad board)
At the start: 2 copper layers, 128 parts, among them U1 ProMicro

Commit message: woooo
Other:
- board text added: "Evelyn Hannah Z.S. Wong"
Changed lines of the file:
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@@
 		(embedded_fonts no)
+	)
+	(gr_text "Evelyn Hannah Z.S. Wong\n"
+		(at 240.50625 46.0375 0)
+		(layer "F.SilkS")
+		(effects
+			(font
+				(size 5 5)
+				(thickness 0.1)
+			)
+			(justify left bottom)
+		)
 	)
 	(segment
@@
 			(pts
 				(arc
-					(start 57.5625 35.71875)
-					(mid 56.148269 36.304504)
-					(end 55.5625 37.71875)
+					(start 341.3125 38.71875)
+					(mid 340.43382 36.59743)
+					(end 338.3125 35.71875)
 				)
 				(arc
-					(start 55.5625 149.60625)
-					(mid 56.148286 151.020464)
-					(end 57.5625 151.60625)
+					(start 56.18125 35.71875)
+					(mid 54.059944 36.597444)
+					(end 53.18125 38.71875)
 				)
 				(arc
-					(start 338.51875 151.60625)
-					(mid 339.932964 151.020464)
-					(end 340.51875 149.60625)
+					(start 53.18125 150.9875)
+					(mid 54.05993 153.10882)
+					(end 56.18125 153.9875)
 				)
 				(arc
-					(start 340.51875 37.71875)
-					(mid 339.932978 36.304522)
-					(end 338.51875 35.71875)
+					(start 338.3125 153.9875)
+					(mid 340.43382 153.10882)
+					(end 341.3125 150.9875)
 				)
 			)
