File: pcb/pcb.kicad_sch (KiCad schematic)
At the start: 0 parts

Commit message: pcbs suck bruh
Parts:
- added C1, C12, C2, C4, C6: 1u, symbol Device:C_Small
- added C10, C11: 22P, symbol Device:C_Small
- added C3: 10u, symbol Device:C_Small
- added C5, C7, C8, C9: 100n, symbol Device:C_Small
- added F1: Fuse_Small, symbol Device:Fuse_Small
- added J1: USB_C_Receptacle_USB2.0_16P, symbol Connector:USB_C_Receptacle_USB2.0_16P
- added J2: Conn_01x04, symbol Connector_Generic:Conn_01x04
- added J3: Conn_01x05, symbol Connector_Generic:Conn_01x05
- added R1, R2, R3: 5.1k, symbol Device:R_Small
- added R4, R5: 27, symbol Device:R_Small
- added R6, R7: 1K, symbol Device:R_Small
- added R8, R9: 5.1K, symbol Device:R_Small
- added SW1, SW2: SW_Push, symbol Switch:SW_Push
- added U1: RP2040, Package_DFN_QFN:QFN-56-1EP_7x7mm_P0.4mm_EP3.2x3.2mm, symbol MCU_RaspberryPi:RP2040
- added U2: XC6206PxxxMR, Package_TO_SOT_SMD:SOT-23-3, symbol Regulator_Linear:XC6206PxxxMR
- added U3: SRV05-4, Package_TO_SOT_SMD:SOT-23-6, symbol Power_Protection:SRV05-4
- added U4: W25Q128JVS, Package_SO:SOIC-8_5.3x5.3mm_P1.27mm, symbol Memory_Flash:W25Q128JVS
- added Y1: Crystal_GND24, symbol Device:Crystal_GND24
Connections:
- new net: R5.2, U1.46 (USB_DM)
- new net: R4.2, U1.47 (USB_DP)
- new net: C3.2, C6.2, C7.2, C8.2, C9.2
- new net: J1.A5 (CC1), R2.1
- new net: J1.B5 (CC2), R1.1
- new net: R7.1, SW2.2
- new net: C10.1, R6.1, Y1.1
- new net: R8.2, R9.1
- new net +1V1: C4.1, C5.1, U1.23 (DVDD), U1.45 (VREG_VOUT), U1.50 (DVDD)
- new net +3V3: C12.1, C2.1, C3.1, C6.1, C7.1, C8.1, C9.1, J3.2 (Pin_2), R3.2, R9.2, U1.1 (IOVDD), U1.10 (IOVDD), U1.22 (IOVDD), U1.33 (IOVDD), U1.42 (IOVDD), U1.43 (ADC_AVDD), U1.44 (VREG_IN), U1.48 (USB_VDD), U1.49 (IOVDD), U2.2 (VO), U4.8 (VCC)
- new net +5V: C1.1, F1.2, J2.1 (Pin_1), U2.3 (VI), U3.5 (VP)
- new net D+: J1.A6 (D+), J1.B6 (D+), J2.3 (Pin_3), R4.1, U3.1 (IO1)
- new net D-: J1.A7 (D-), J1.B7 (D-), J2.2 (Pin_2), R5.1, U3.3 (IO2)
- new net GND: C1.2, C10.2, C11.2, C12.2, C2.2, C4.2, C5.2, J1.A1 (GND), J1.A12 (GND), J1.B1 (GND), J1.B12 (GND), J1.S1 (SHIELD), J2.4 (Pin_4), J3.3 (Pin_3), R1.2, R2.2, SW1.1, SW2.1, U1.19 (TESTEN), U1.57 (GND), U2.1 (GND), U3.2 (VN), U4.4 (GND), Y1.2, Y1.4
- new net Q100: U1.53 (QSPI_SD0), U4.5 (DI/IO_{0})
- new net Q101: U1.55 (QSPI_SD1), U4.2 (DO/IO_{1})
- new net Q102: U1.54 (QSPI_SD2), U4.3 (~{WP}/IO_{2})
- new net Q103: U1.51 (QSPI_SD3), U4.7 (~{HOLD}/~{RESET}/IO_{3})
- new net QCLK: U1.52 (QSPI_SCLK), U4.6 (CLK)
- new net QSEL: R7.2, R8.1, U1.56 (QSPI_SS), U4.1 (~{CS})
- new net RESET: J3.1 (Pin_1), R3.1, SW1.2, U1.26 (RUN)
- new net SWC: J3.4 (Pin_4), U1.24 (SWCLK)
- new net SWD: J3.5 (Pin_5), U1.25 (SWD)
- new net VBUS: F1.1, J1.A4 (VBUS), J1.A9 (VBUS), J1.B4 (VBUS), J1.B9 (VBUS)
- new net XIN: C11.1, U1.20 (XIN), Y1.3
- new net XOUT: R6.2, U1.21 (XOUT)
- no-connect marks 0 -> 4

Commit message: sob
Parts:
- added D1, D10, D11, D12, D13, D14, D15, D16, D17, D18, D19, D2, D20, D21, D22, D23, D24, D25, D26, D27, D28, D29, D3, D30, D31, D32, D33, D34, D35, D36, D37, D38, D39, D4, D40, D41, D42, D43, D44, D45, D46, D47, D48, D49, D5, D50, D51, D52, D53, D54, D55, D56, D57, D58, D59, D6, D60, D61, D62, D63, D64, D65, D66, D67, D68, D69, D7, D70, D71, D72, D73, D74, D75, D76, D77, D78, D79, D8, D80, D81, D82, D83, D84, D9: D_Small, Diode_SMD:D_SOD-123, symbol Device:D_Small
- added MX1, MX10, MX11, MX12, MX13, MX14, MX15, MX16, MX17, MX18, MX19, MX2, MX20, MX21, MX22, MX23, MX24, MX25, MX26, MX27, MX28, MX29, MX3, MX30, MX32, MX33, MX34, MX35, MX36, MX37, MX38, MX39, MX4, MX40, MX41, MX42, MX43, MX45, MX46, MX47, MX49, MX5, MX50, MX51, MX52, MX53, MX54, MX55, MX56, MX57, MX58, MX59, MX6, MX60, MX61, MX62, MX63, MX64, MX65, MX66, MX67, MX68, MX69, MX7, MX70, MX71, MX72, MX73, MX77, MX8, MX82, MX83, MX84, MX9: MX_SW_solder, PCM_marbastlib-mx:SW_MX_1u, symbol PCM_marbastlib-mx:MX_SW_solder
- added MX31, MX44: MX_SW_solder, PCM_marbastlib-mx:SW_MX_1.5u, symbol PCM_marbastlib-mx:MX_SW_solder
- added MX48: MX_SW_solder, PCM_marbastlib-mx:SW_MX_1.75u, symbol PCM_marbastlib-mx:MX_SW_solder
- added MX74, MX75, MX76, MX78, MX79, MX80, MX81: MX_SW_solder, PCM_marbastlib-mx:SW_MX_1.25u, symbol PCM_marbastlib-mx:MX_SW_solder
- added S1: MX_stab, PCM_marbastlib-mx:STAB_MX_P_6.25u, symbol PCM_marbastlib-mx:MX_stab
- added S2, S3, S4, S5: MX_stab, PCM_marbastlib-mx:STAB_MX_P_2u, symbol PCM_marbastlib-mx:MX_stab
- BOOT1: renamed from SW2; footprint (none) -> Button_Switch_SMD:SW_SPST_TL3342
- C1, C11, C2, C6, C7, C8, C9: footprint (none) -> Capacitor_SMD:C_0402_1005Metric
- C10: renamed from C12; footprint (none) -> Capacitor_SMD:C_0402_1005Metric
- C12: renamed from C10; footprint (none) -> Capacitor_SMD:C_0402_1005Metric
- C3: renamed from C4; footprint (none) -> Capacitor_SMD:C_0402_1005Metric
- C4: renamed from C5; footprint (none) -> Capacitor_SMD:C_0402_1005Metric
- C5: renamed from C3; footprint (none) -> Capacitor_SMD:C_0603_1608Metric
- F1: footprint (none) -> Fuse:Fuse_1206_3216Metric
- J1: footprint (none) -> Connector_USB:USB_C_Receptacle_HRO_TYPE-C-31-M-12
- J2: footprint (none) -> Connector_JST:JST_SH_SM04B-SRSS-TB_1x04-1MP_P1.00mm_Horizontal
- J3: footprint (none) -> Connector_PinHeader_2.54mm:PinHeader_1x05_P2.54mm_Vertical
- R1: renamed from R2; footprint (none) -> Resistor_SMD:R_0402_1005Metric
- R2: renamed from R1; footprint (none) -> Resistor_SMD:R_0402_1005Metric
- R3: renamed from R9; footprint (none) -> Resistor_SMD:R_0402_1005Metric
- R4: renamed from R8; footprint (none) -> Resistor_SMD:R_0402_1005Metric
- R5: renamed from R3; footprint (none) -> Resistor_SMD:R_0402_1005Metric
- R6: renamed from R7; footprint (none) -> Resistor_SMD:R_0402_1005Metric
- R7: renamed from R4; footprint (none) -> Resistor_SMD:R_0402_1005Metric
- R8: renamed from R5; footprint (none) -> Resistor_SMD:R_0402_1005Metric
- R9: renamed from R6; footprint (none) -> Resistor_SMD:R_0402_1005Metric
- RST1: renamed from SW1; footprint (none) -> Button_Switch_SMD:SW_SPST_TL3342
- Y1: footprint (none) -> Crystal:Crystal_SMD_3225-4Pin_3.2x2.5mm
- renumbered U2 to U1, U3 to U2, U1 to U3
Connections:
- new net: D65.2 (A), MX65.2
- new net: D54.2 (A), MX54.2
- new net: D60.2 (A), MX60.2
- new net: D71.2 (A), MX71.2
- new net: D48.2 (A), MX48.2
- new net: D7.2 (A), MX7.2
- new net: D36.2 (A), MX36.2
- new net: D31.2 (A), MX31.2
- new net: D64.2 (A), MX64.2
- new net: D52.2 (A), MX52.2
- new net: D72.2 (A), MX72.2
- new net: D79.2 (A), MX79.2
- new net: D51.2 (A), MX51.2
- new net: D43.2 (A), MX43.2
- new net: D17.2 (A), MX17.2
- new net: D70.2 (A), MX70.2
- new net: D55.2 (A), MX55.2
- new net: D69.2 (A), MX69.2
- new net: D37.2 (A), MX37.2
- new net: D4.2 (A), MX4.2
- new net: D68.2 (A), MX68.2
- new net: D67.2 (A), MX67.2
- new net: D26.2 (A), MX26.2
- new net: D66.2 (A), MX66.2
- new net: D15.2 (A), MX15.2
- new net: D33.2 (A), MX33.2
- new net: D19.2 (A), MX19.2
- new net: D22.2 (A), MX22.2
- new net: D62.2 (A), MX62.2
- new net: D45.2 (A), MX45.2
- new net: D6.2 (A), MX6.2
- new net: D28.2 (A), MX28.2
- new net: D83.2 (A), MX83.2
- new net: D20.2 (A), MX20.2
- new net: D59.2 (A), MX59.2
- new net: D57.2 (A), MX57.2
- new net: D84.2 (A), MX84.2
- new net: D76.2 (A), MX76.2
- new net: D73.2 (A), MX73.2
- new net: D50.2 (A), MX50.2
- new net: D14.2 (A), MX14.2
- new net: D74.2 (A), MX74.2
- new net: D53.2 (A), MX53.2
- new net: D58.2 (A), MX58.2
- new net: D49.2 (A), MX49.2
- new net: D11.2 (A), MX11.2
- new net: D9.2 (A), MX9.2
- new net: D80.2 (A), MX80.2
- new net: D18.2 (A), MX18.2
- new net: D16.2 (A), MX16.2
- new net: D56.2 (A), MX56.2
- new net: D25.2 (A), MX25.2
- new net: D44.2 (A), MX44.2
- new net: D78.2 (A), MX78.2
- new net: D42.2 (A), MX42.2
- new net: D30.2 (A), MX30.2
- new net: D61.2 (A), MX61.2
- new net: D21.2 (A), MX21.2
- new net: D77.2 (A), MX77.2
- new net: D2.2 (A), MX2.2
- new net: D34.2 (A), MX34.2
- new net: D5.2 (A), MX5.2
- new net: D40.2 (A), MX40.2
- new net: D63.2 (A), MX63.2
- new net: D41.2 (A), MX41.2
- new net: D8.2 (A), MX8.2
- new net: D23.2 (A), MX23.2
- new net: D32.2 (A), MX32.2
- new net: D29.2 (A), MX29.2
- new net: D81.2 (A), MX81.2
- new net: D1.2 (A), MX1.2
- new net: D38.2 (A), MX38.2
- new net: D39.2 (A), MX39.2
- new net: D46.2 (A), MX46.2
- new net: D27.2 (A), MX27.2
- new net: D13.2 (A), MX13.2
- new net: D24.2 (A), MX24.2
- new net: D75.2 (A), MX75.2
- new net: D47.2 (A), MX47.2
- new net: D3.2 (A), MX3.2
- new net: D12.2 (A), MX12.2
- new net: D35.2 (A), MX35.2
- new net: D82.2 (A), MX82.2
- new net: D10.2 (A), MX10.2
Other:
- moved on the sheet: C11, C12, R9, Y1

Commit message: sob
Connections:
- net D-: now also U2.6 (IO4); no longer U2.3 (IO2)
- no-connect marks 4 -> 5
Changed lines of the file:
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@@
+	)
+	(no_connect
+		(at 77.47 68.58)
 	)
 	(no_connect
@@
 	(global_label "D-"
 		(shape input)
-		(at 77.47 68.58 180)
+		(at 102.87 68.58 0)
 		(fields_autoplaced yes)
 		(effects
@@
 				(size 1.27 1.27)
 			)
-			(justify right)
+			(justify left)
 		)
 		(property "Intersheetrefs" "${INTERSHEET_REFS}"
-			(at 71.6424 68.58 0)
+			(at 108.6976 68.58 0)
 			(effects
 				(font
 					(size 1.27 1.27)
 				)
-				(justify right)
+				(justify left)
 				(hide yes)
 			)

Commit message: ahhhhhhhhhhhhhh
Parts:
- removed BOOT1, RST1: SW_Push, Button_Switch_SMD:SW_SPST_TL3342, symbol Switch:SW_Push
- removed C1, C10, C2, C3, C6: 1u, Capacitor_SMD:C_0402_1005Metric, symbol Device:C_Small
- removed C11, C12: 22P, Capacitor_SMD:C_0402_1005Metric, symbol Device:C_Small
- removed C4, C7, C8, C9: 100n, Capacitor_SMD:C_0402_1005Metric, symbol Device:C_Small
- removed C5: 10u, Capacitor_SMD:C_0603_1608Metric, symbol Device:C_Small
- removed D28, D29, D30, D45, D46, D47, D73, D82, D83, D84: D_Small, Diode_SMD:D_SOD-123, symbol Device:D_Small
- removed F1: Fuse_Small, Fuse:Fuse_1206_3216Metric, symbol Device:Fuse_Small
- removed J1: USB_C_Receptacle_USB2.0_16P, Connector_USB:USB_C_Receptacle_HRO_TYPE-C-31-M-12, symbol Connector:USB_C_Receptacle_USB2.0_16P
- removed J2: Conn_01x04, Connector_JST:JST_SH_SM04B-SRSS-TB_1x04-1MP_P1.00mm_Horizontal, symbol Connector_Generic:Conn_01x04
- removed J3: Conn_01x05, Connector_PinHeader_2.54mm:PinHeader_1x05_P2.54mm_Vertical, symbol Connector_Generic:Conn_01x05
- removed MX28, MX29, MX30, MX45, MX46, MX47, MX73, MX82, MX83, MX84: MX_SW_solder, PCM_marbastlib-mx:SW_MX_1u, symbol PCM_marbastlib-mx:MX_SW_solder
- removed R1, R2, R5: 5.1k, Resistor_SMD:R_0402_1005Metric, symbol Device:R_Small
- removed R3, R4: 5.1K, Resistor_SMD:R_0402_1005Metric, symbol Device:R_Small
- removed R6, R9: 1K, Resistor_SMD:R_0402_1005Metric, symbol Device:R_Small
- removed R7, R8: 27, Resistor_SMD:R_0402_1005Metric, symbol Device:R_Small
- removed U1: XC6206PxxxMR, Package_TO_SOT_SMD:SOT-23-3, symbol Regulator_Linear:XC6206PxxxMR
- removed U2: SRV05-4, Package_TO_SOT_SMD:SOT-23-6, symbol Power_Protection:SRV05-4
- removed U3: RP2040, Package_DFN_QFN:QFN-56-1EP_7x7mm_P0.4mm_EP3.2x3.2mm, symbol MCU_RaspberryPi:RP2040
- removed U4: W25Q128JVS, Package_SO:SOIC-8_5.3x5.3mm_P1.27mm, symbol Memory_Flash:W25Q128JVS
- removed Y1: Crystal_GND24, Crystal:Crystal_SMD_3225-4Pin_3.2x2.5mm, symbol Device:Crystal_GND24
Connections:
- net at D65.1 (K): now also D61.1 (K), D62.1 (K), D63.1 (K), D64.1 (K), D66.1 (K), D67.1 (K), D68.1 (K), D69.1 (K), D70.1 (K), D71.1 (K), D72.1 (K)
- net COL6: now reaches MX54.1
- net COL6: now also MX20.1, MX37.1, MX6.1, MX66.1, MX77.1
- net COL12: now reaches MX60.1
- net COL12: now also MX12.1, MX26.1, MX43.1, MX72.1, MX81.1
- net COL1: now reaches MX48.1
- net COL1: now also MX1.1, MX14.1, MX31.1, MX74.1
- net COL7: now reaches MX7.1
- net COL7: now also MX21.1, MX38.1, MX55.1, MX67.1
- net COL5: now reaches MX36.1
- net COL5: now also MX19.1, MX5.1, MX53.1, MX65.1
- net at D31.1 (K): now also D32.1 (K), D33.1 (K), D34.1 (K), D35.1 (K), D36.1 (K), D37.1 (K), D38.1 (K), D39.1 (K), D40.1 (K), D41.1 (K), D42.1 (K), D43.1 (K), D44.1 (K)
- net at D52.1 (K): now also D48.1 (K), D49.1 (K), D50.1 (K), D51.1 (K), D53.1 (K), D54.1 (K), D55.1 (K), D56.1 (K), D57.1 (K), D58.1 (K), D59.1 (K), D60.1 (K)
- net COL10: now reaches MX79.1
- net COL10: now also MX10.1, MX24.1, MX41.1, MX58.1, MX70.1
- net COL3: now reaches MX51.1
- net COL3: now also MX17.1, MX3.1, MX34.1, MX63.1, MX76.1
- net at D4.1 (K): now also D1.1 (K), D10.1 (K), D11.1 (K), D12.1 (K), D13.1 (K), D2.1 (K), D3.1 (K), D5.1 (K), D6.1 (K), D7.1 (K), D8.1 (K), D9.1 (K)
- net at D15.1 (K): now also D14.1 (K), D16.1 (K), D17.1 (K), D18.1 (K), D19.1 (K), D20.1 (K), D21.1 (K), D22.1 (K), D23.1 (K), D24.1 (K), D25.1 (K), D26.1 (K), D27.1 (K)
- net COL8: now reaches MX22.1
- net COL8: now also MX39.1, MX56.1, MX68.1, MX8.1
- net COL2: now reaches MX62.1
- net COL2: now also MX16.1, MX2.1, MX33.1, MX50.1, MX75.1
- net COL11: now reaches MX59.1
- net COL11: now also MX11.1, MX25.1, MX42.1, MX71.1, MX80.1
- net at MX15.1: now also MX32.1, MX49.1, MX61.1
- net at D80.1 (K): now also D74.1 (K), D75.1 (K), D76.1 (K), D77.1 (K), D78.1 (K), D79.1 (K), D81.1 (K)
- net COL4: now reaches MX18.1
- net COL4: now also MX35.1, MX4.1, MX52.1, MX64.1
- net COL13: now reaches MX44.1
- net COL13: now also MX13.1, MX27.1
- net COL9: now reaches MX57.1
- net COL9: now also MX23.1, MX40.1, MX69.1, MX78.1, MX9.1
- no-connect marks 5 -> 1
Other:
- moved on the sheet: D1, D10, D11, D12, D13, D14, D15, D16, D17, D18, D19, D2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

Commit message: woooo
Parts:
- removed D1, D10, D11, D12, D13, D2, D3, D4, D5, D6, D7, D8, D9: D_Small, Diode_SMD:D_SOD-123, symbol Device:D_Small
- removed MX1, MX10, MX11, MX12, MX13, MX2, MX3, MX4, MX5, MX6, MX7, MX8, MX9: MX_SW_solder, PCM_marbastlib-mx:SW_MX_1u, symbol PCM_marbastlib-mx:MX_SW_solder
- added U1: ProMicro, PCM_marbastlib-xp-promicroish:ProMicro_USBup, symbol PCM_marbastlib-promicroish:Arduino_ProMicro
- renumbered D14 to D1, D23 to D10, D24 to D11, D25 to D12, D26 to D13, D27 to D14, D31 to D15, D32 to D16, D33 to D17, D34 to D18, D35 to D19, D15 to D2, D36 to D20, D37 to D21, D38 to D22, D39 to D23, D40 to D24, D41 to D25, D42 to D26, D43 to D27, D44 to D28, D48 to D29, D16 to D3, D49 to D30, D50 to D31, D51 to D32, D52 to D33, D53 to D34, D54 to D35, D55 to D36, D56 to D37, D57 to D38, D58 to D39, D17 to D4, D59 to D40, D60 to D41, D61 to D42, D62 to D43, D63 to D44, D64 to D45, D65 to D46, D66 to D47, D67 to D48, D68 to D49, D18 to D5, D69 to D50, D70 to D51, D71 to D52, D72 to D53, D74 to D54, D75 to D55, D76 to D56, D77 to D57, D78 to D58, D79 to D59, D19 to D6, D80 to D60, D81 to D61, D20 to D7, D21 to D8, D22 to D9, MX14 to MX1, MX23 to MX10, MX24 to MX11, MX25 to MX12, MX26 to MX13, MX27 to MX14, MX31 to MX15, MX32 to MX16, MX33 to MX17, MX34 to MX18, MX35 to MX19, MX15 to MX2, MX36 to MX20, MX37 to MX21, MX38 to MX22, MX39 to MX23, MX40 to MX24, MX41 to MX25, MX42 to MX26, MX43 to MX27, MX44 to MX28, MX48 to MX29, MX16 to MX3, MX49 to MX30, MX50 to MX31, MX51 to MX32, MX52 to MX33, MX53 to MX34, MX54 to MX35, MX55 to MX36, MX56 to MX37, MX57 to MX38, MX58 to MX39, MX17 to MX4, MX59 to MX40, MX60 to MX41, MX61 to MX42, MX62 to MX43, MX63 to MX44, MX64 to MX45, MX65 to MX46, MX66 to MX47, MX67 to MX48, MX68 to MX49, MX18 to MX5, MX69 to MX50, MX70 to MX51, MX71 to MX52, MX72 to MX53, MX74 to MX54, MX75 to MX55, MX76 to MX56, MX77 to MX57, MX78 to MX58, MX79 to MX59, MX19 to MX6, MX80 to MX60, MX81 to MX61, MX20 to MX7, MX21 to MX8, MX22 to MX9, S5 to S1, S4 to S2, S2 to S3, S3 to S4, S1 to S5
Connections:
- net COL1: now also U1.2 (D2-RX)
- net COL10: now also U1.17 (F4)
- net COL11: now also U1.18 (F5)
- net COL12: now also U1.19 (F6)
- net COL13: now also U1.20 (F7)
- net COL2: now also U1.5 (D1)
- net COL3: now also U1.6 (D0)
- net COL4: now also U1.7 (D4)
- net COL5: now also U1.8 (C6)
- net COL6: now also U1.9 (D7)
- net COL7: now also U1.10 (E6)
- net COL8: now also U1.11 (B4)
- net COL9: now also U1.12 (B5)
- net ROW4: now reaches D42.1 (K), D43.1 (K), D44.1 (K), D45.1 (K), D46.1 (K), D47.1 (K), D48.1 (K), D49.1 (K), D50.1 (K), D51.1 (K), D52.1 (K), D53.1 (K)
- net ROW4: now also U1.23 (B2)
- net ROW2: now reaches D15.1 (K), D16.1 (K), D17.1 (K), D18.1 (K), D19.1 (K), D20.1 (K), D21.1 (K), D22.1 (K), D23.1 (K), D24.1 (K), D25.1 (K), D26.1 (K), D27.1 (K), D28.1 (K)
- net ROW2: now also U1.21 (B1)
- net ROW3: now reaches D29.1 (K), D30.1 (K), D31.1 (K), D32.1 (K), D33.1 (K), D34.1 (K), D35.1 (K), D36.1 (K), D37.1 (K), D38.1 (K), D39.1 (K), D40.1 (K), D41.1 (K)
- net ROW3: now also U1.22 (B3)
- net ROW1: now reaches D1.1 (K), D10.1 (K), D11.1 (K), D12.1 (K), D13.1 (K), D14.1 (K), D2.1 (K), D3.1 (K), D4.1 (K), D5.1 (K), D6.1 (K), D7.1 (K), D8.1 (K), D9.1 (K)
- net ROW1: now also U1.1 (D3-TX)
- net COL14: now reaches MX16.1, MX2.1, MX30.1, MX42.1
- net COL14: now also U1.13 (B0)
- net ROW5: now reaches D54.1 (K), D55.1 (K), D56.1 (K), D57.1 (K), D58.1 (K), D59.1 (K), D60.1 (K), D61.1 (K)
- net ROW5: now also U1.24 (B6)
- new net GND: U1.14 (GND), U1.3 (GND), U1.4 (GND)
- no-connect marks 1 -> 2
Other:
- moved on the sheet: S1
