File: pcb/pcb.kicad_pcb (KiCad board)
At the start: 2 copper layers, 128 parts, among them U1 ProMicro

Commit message: fml!
Other:
- board text added: "Evelyn Hannah Z.S. Wong"
Changed lines of the file:
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@@
 		(embedded_fonts no)
+	)
+	(gr_text "Evelyn Hannah Z.S. Wong\n"
+		(at 240.50625 46.0375 0)
+		(layer "F.SilkS")
+		(effects
+			(font
+				(size 5 5)
+				(thickness 0.1)
+			)
+			(justify left bottom)
+		)
 	)
 	(segment
@@
 			(pts
 				(arc
-					(start 57.5625 35.71875)
-					(mid 56.148269 36.304504)
-					(end 55.5625 37.71875)
+					(start 341.3125 38.71875)
+					(mid 340.43382 36.59743)
+					(end 338.3125 35.71875)
 				)
 				(arc
-					(start 55.5625 149.60625)
-					(mid 56.148286 151.020464)
-					(end 57.5625 151.60625)
+					(start 56.18125 35.71875)
+					(mid 54.059944 36.597444)
+					(end 53.18125 38.71875)
 				)
 				(arc
-					(start 338.51875 151.60625)
-					(mid 339.932964 151.020464)
-					(end 340.51875 149.60625)
+					(start 53.18125 150.9875)
+					(mid 54.05993 153.10882)
+					(end 56.18125 153.9875)
 				)
 				(arc
-					(start 340.51875 37.71875)
-					(mid 339.932978 36.304522)
-					(end 338.51875 35.71875)
+					(start 338.3125 153.9875)
+					(mid 340.43382 153.10882)
+					(end 341.3125 150.9875)
 				)
 			)

Commit message: FML
Parts:
- D1, D10, D11, D12, D13, D14, D15, D16, D17, D18, D19, D2, D20, D21, D22, D23, D24, D25, D26, D27, D28, D29, D3, D30, D31, D32, D33, D34, D35, D36, D37, D38, D39, D4, D40, D41, D42, D43, D44, D45, D46, D47, D48, D49, D5, D50, D51, D52, D53, D54, D55, D56, D57, D58, D59, D6, D60, D61, D7, D8, D9: moved to B.Cu
- moved S1 43.4 mm to (37.3, 106.3), turned to 180 degrees
- moved S3 43.4 mm to (280.2, 87.3), turned to 180 degrees
- moved MX20 43.4 mm to (130.2, 68.2)
- moved MX25 43.4 mm to (225.4, 68.2)
- moved MX26 43.4 mm to (244.5, 68.2)
- moved MX35 43.4 mm to (154.0, 87.3)
- moved MX40 43.4 mm to (249.2, 87.3)
- moved MX50 43.4 mm to (201.6, 106.3)
- moved MX51 43.4 mm to (220.7, 106.3)
- moved MX9 43.4 mm to (177.8, 49.2)
- moved MX2 43.4 mm to (44.4, 49.2)
- moved MX29 43.4 mm to (32.5, 87.3)
- moved MX3 43.4 mm to (63.5, 49.2)
- moved MX42 43.4 mm to (37.3, 106.3)
- moved MX55 43.4 mm to (51.6, 125.4)
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Connections:
- D1 pad 1: ROW1 -> ROW0
- D10 pad 1: ROW1 -> ROW0
- D11 pad 1: ROW1 -> ROW0
- D12 pad 1: ROW1 -> ROW0
- D13 pad 1: ROW1 -> ROW0
- D14 pad 1: ROW1 -> ROW0
- D15 pad 1: ROW2 -> ROW1
- D16 pad 1: ROW2 -> ROW1
- D17 pad 1: ROW2 -> ROW1
- D18 pad 1: ROW2 -> ROW1
- D19 pad 1: ROW2 -> ROW1
- D2 pad 1: ROW1 -> ROW0
- D20 pad 1: ROW2 -> ROW1
- D21 pad 1: ROW2 -> ROW1
- D22 pad 1: ROW2 -> ROW1
- D23 pad 1: ROW2 -> ROW1
- D24 pad 1: ROW2 -> ROW1
- D25 pad 1: ROW2 -> ROW1
- D26 pad 1: ROW2 -> ROW1
- D27 pad 1: ROW2 -> ROW1
- D28 pad 1: ROW2 -> ROW1
- D29 pad 1: ROW3 -> ROW2
- D3 pad 1: ROW1 -> ROW0
- D30 pad 1: ROW3 -> ROW2
- D31 pad 1: ROW3 -> ROW2
- D32 pad 1: ROW3 -> ROW2
- D33 pad 1: ROW3 -> ROW2
- D34 pad 1: ROW3 -> ROW2
- D35 pad 1: ROW3 -> ROW2
- D36 pad 1: ROW3 -> ROW2
- D37 pad 1: ROW3 -> ROW2
- D38 pad 1: ROW3 -> ROW2
- D39 pad 1: ROW3 -> ROW2
- D4 pad 1: ROW1 -> ROW0
- D40 pad 1: ROW3 -> ROW2
- D41 pad 1: ROW3 -> ROW2
- D42 pad 1: ROW4 -> ROW3
- D43 pad 1: ROW4 -> ROW3
- D44 pad 1: ROW4 -> ROW3
- D45 pad 1: ROW4 -> ROW3
- D46 pad 1: ROW4 -> ROW3
- D47 pad 1: ROW4 -> ROW3
- D48 pad 1: ROW4 -> ROW3
- D49 pad 1: ROW4 -> ROW3
- D5 pad 1: ROW1 -> ROW0
- D50 pad 1: ROW4 -> ROW3
- D51 pad 1: ROW4 -> ROW3
- D52 pad 1: ROW4 -> ROW3
- D53 pad 1: ROW4 -> ROW3
- D54 pad 1: ROW5 -> ROW4
- D55 pad 1: ROW5 -> ROW4
- D56 pad 1: ROW5 -> ROW4
- D57 pad 1: ROW5 -> ROW4
- D58 pad 1: ROW5 -> ROW4
- D59 pad 1: ROW5 -> ROW4
- D6 pad 1: ROW1 -> ROW0
- D60 pad 1: ROW5 -> ROW4
- D61 pad 1: ROW5 -> ROW4
- D7 pad 1: ROW1 -> ROW0
- D8 pad 1: ROW1 -> ROW0
- D9 pad 1: ROW1 -> ROW0
- MX1 pad 1: COL1 -> COL0
- MX15 pad 1: COL1 -> COL0
- MX16 pad 1: COL14 -> COL1
- MX2 pad 1: COL14 -> COL1
- MX29 pad 1: COL1 -> COL0
- MX30 pad 1: COL14 -> COL1
- MX42 pad 1: COL14 -> COL1
- MX54 pad 1: COL1 -> COL0
- U1 pad 1: ROW1 -> ROW0
- U1 pad 10: COL7 -> COL6
- U1 pad 11: COL8 -> COL7
- U1 pad 12: COL9 -> COL8
- U1 pad 13: COL14 -> COL9
- U1 pad 2: COL1 -> COL0
- U1 pad 21: ROW2 -> ROW4
- U1 pad 23: ROW4 -> ROW2
- U1 pad 24: ROW5 -> ROW1
- U1 pad 5: COL2 -> COL1
- U1 pad 6: COL3 -> COL2
- U1 pad 7: COL4 -> COL3
- U1 pad 8: COL5 -> COL4
- U1 pad 9: COL6 -> COL5
Routing:
- net ROW5: track 619.1 -> 0.00 mm
- net ROW0: track 0.00 -> 279.3 mm
- net ROW3: track 572.9 -> 362.3 mm
- net ROW2: track 559.0 -> 351.3 mm
- net ROW4: track 583.9 -> 397.0 mm
- net COL14: track 113.8 -> 0.00 mm
- net COL0: track 0.00 -> 91.0 mm
- net ROW1: track 283.0 -> 343.2 mm
- net COL9: track 243.1 -> 280.8 mm
- net COL7: track 185.3 -> 179.8 mm
- net COL8: track 201.6 -> 196.3 mm
- net COL6: track 188.9 -> 183.8 mm
- net COL3: track 143.8 -> 138.7 mm
- net COL5: track 152.5 -> 147.6 mm
- net COL4: track 136.2 -> 131.5 mm
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Other:
- board outline added: 285.8 x 114.3 mm

Commit message: sleep
Parts:
- removed U1: ProMicro, PCM_marbastlib-xp-promicroish:ProMicro_USBup
- added J1: USB_C_Receptacle_USB2.0_16P, Connector_USB:USB_C_Receptacle_HRO_TYPE-C-31-M-12, F.Cu at (88.1, 130.2)
- added R1: 5.1k, Resistor_SMD:R_0402_1005Metric, F.Cu at (86.2, 123.8)
- added R2: 5.1k, Resistor_SMD:R_0402_1005Metric, F.Cu at (90.8, 123.8)
- added RST1: SW_Push, Button_Switch_SMD:SW_SPST_TL3305B, F.Cu at (119.9, 123.8)
- added U3: Elite-C, PCM_marbastlib-xp-promicroish:Elite-C_ACH, F.Cu at (174.6, 123.0)
Routing:
- net COL0: track 91.0 -> 265.1 mm
- net COL9: track 280.8 -> 136.9 mm, vias 0 -> 2
- net COL10: track 294.2 -> 152.5 mm, vias 0 -> 2
- net COL1: track 90.3 -> 231.5 mm, vias 0 -> 2
- net COL11: track 316.1 -> 196.1 mm, vias 0 -> 2
- net ROW3: track 362.3 -> 244.8 mm
- net COL12: track 325.0 -> 219.5 mm, vias 0 -> 2
- net GND: track 18.8 -> 121.8 mm
- net COL2: track 126.2 -> 225.8 mm, vias 0 -> 2
- net COL8: track 196.3 -> 97.9 mm
- net ROW4: track 397.0 -> 303.8 mm, vias 0 -> 2
- net VBUS: track 0.00 -> 85.6 mm, vias 0 -> 4
- net D-: track 0.00 -> 83.4 mm, vias 0 -> 2
- net D+: track 0.00 -> 78.0 mm, vias 0 -> 2
- net ROW2: track 351.3 -> 275.0 mm, vias 0 -> 2
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Other:
- board size 285.8 x 114.3 mm -> 287.3 x 96.8 mm
