File: messups!/pcb/pcb.kicad_sch (KiCad schematic)
At the start: 128 parts, among them U1 ProMicro

Commit message: FML
Connections:
- net COL0 is gone; now on net COL1: MX1.1, MX15.1, MX29.1, MX54.1, U1.2 (D2-RX)
- net ROW0 is gone; now on net ROW1: D1.1 (K), D10.1 (K), D11.1 (K), D12.1 (K), D13.1 (K), D14.1 (K), D2.1 (K), D3.1 (K), D4.1 (K), D5.1 (K), D6.1 (K), D7.1 (K), D8.1 (K), D9.1 (K), U1.1 (D3-TX)
- net COL1: no longer MX16.1, MX2.1, MX30.1, MX42.1, U1.5 (D1)
- net COL2: now also U1.5 (D1); no longer U1.6 (D0)
- net COL3: now also U1.6 (D0); no longer U1.7 (D4)
- net COL4: now also U1.7 (D4); no longer U1.8 (C6)
- net COL5: now also U1.8 (C6); no longer U1.9 (D7)
- net COL6: now also U1.9 (D7); no longer U1.10 (E6)
- net COL7: now also U1.10 (E6); no longer U1.11 (B4)
- net COL8: now also U1.11 (B4); no longer U1.12 (B5)
- net COL9: now also U1.12 (B5); no longer U1.13 (B0)
- net ROW1: no longer D15.1 (K), D16.1 (K), D17.1 (K), D18.1 (K), D19.1 (K), D20.1 (K), D21.1 (K), D22.1 (K), D23.1 (K), D24.1 (K), D25.1 (K), D26.1 (K), D27.1 (K), D28.1 (K), U1.24 (B6)
- net ROW2: now also D15.1 (K), D16.1 (K), D17.1 (K), D18.1 (K), D19.1 (K), D20.1 (K), D21.1 (K), D22.1 (K), D23.1 (K), D24.1 (K), D25.1 (K), D26.1 (K), D27.1 (K), D28.1 (K), U1.21 (B1); no longer D29.1 (K), D30.1 (K), D31.1 (K), D32.1 (K), D33.1 (K), D34.1 (K), D35.1 (K), D36.1 (K), D37.1 (K), D38.1 (K), D39.1 (K), D40.1 (K), D41.1 (K), U1.23 (B2)
- net ROW3: now also D29.1 (K), D30.1 (K), D31.1 (K), D32.1 (K), D33.1 (K), D34.1 (K), D35.1 (K), D36.1 (K), D37.1 (K), D38.1 (K), D39.1 (K), D40.1 (K), D41.1 (K); no longer D42.1 (K), D43.1 (K), D44.1 (K), D45.1 (K), D46.1 (K), D47.1 (K), D48.1 (K), D49.1 (K), D50.1 (K), D51.1 (K), D52.1 (K), D53.1 (K)
- net ROW4: now also D42.1 (K), D43.1 (K), D44.1 (K), D45.1 (K), D46.1 (K), D47.1 (K), D48.1 (K), D49.1 (K), D50.1 (K), D51.1 (K), D52.1 (K), D53.1 (K), U1.23 (B2); no longer D54.1 (K), D55.1 (K), D56.1 (K), D57.1 (K), D58.1 (K), D59.1 (K), D60.1 (K), D61.1 (K), U1.21 (B1)
- new net COL14: MX16.1, MX2.1, MX30.1, MX42.1, U1.13 (B0)
- new net ROW5: D54.1 (K), D55.1 (K), D56.1 (K), D57.1 (K), D58.1 (K), D59.1 (K), D60.1 (K), D61.1 (K), U1.24 (B6)
Other:
- moved on the sheet: D1, D10, D11, D12, D13, D14, D15, D16, D17, D18, D19, D2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
